File: BLDC_Testboard/BLDC_Testboard.kicad_sch (KiCad schematic)
At the start: 34 parts, among them J1 Conn_ARM_JTAG_SWD_10, P1 USB_C_Plug_USB2.0, U1 STM32G491CCUx, U2 LT1963AxST-3.3, U3 ADP2302ARDZ-3.3

Commit message: Add files via upload
Parts:
- removed C11: 600u, Capacitor_SMD:C_Elec_3x5.4, symbol Device:C
- added C11, C27, C28, C30: 100u, Capacitor_SMD:CP_Elec_3x5.3, symbol Device:C_Polarized
- added C29, C31, C32, C33: 10n, Capacitor_SMD:C_0201_0603Metric, symbol Device:C_Small
- added D4: SD36_SOD323, Diode_SMD:D_SOD-323, symbol Diode:SD36_SOD323
- added J5: Conn_01x02_Pin, Connector_PinHeader_1.00mm:PinHeader_1x02_P1.00mm_Vertical, symbol Connector:Conn_01x02_Pin
- added L3: 1u, Inductor_SMD:L_0201_0603Metric, symbol Device:L
- added Q7: Si7617DN, Package_SO:Vishay_PowerPAK_1212-8_Single, symbol Transistor_FET:Si7617DN
- added X1: 32MHz, Crystal:Crystal_SMD_2012-2Pin_2.0x1.2mm_HandSoldering, symbol Device:Crystal
- added X2: 32kHz, Crystal:Crystal_SMD_2012-2Pin_2.0x1.2mm_HandSoldering, symbol Device:Crystal
- BAT_+1: renamed from U_Bat+; value U_Bat + -> BAT_IN; footprint (none) -> Connector_Wire:SolderWire-2.5sqmm_1x01_D2.4mm_OD4.4mm
- BAT_-1: renamed from U_Bat-; value U_Bat - -> BAT_OUT; footprint (none) -> Connector_Wire:SolderWire-2.5sqmm_1x01_D2.4mm_OD4.4mm
- C1, C10, C2, C24, C25, C26, C3, C4, C5, C6, C7, C8, C9, C_OUT_1, C_OUT_2: footprint (none) -> Capacitor_SMD:C_0201_0603Metric
- C_BST1: renamed from C_BST; footprint (none) -> Capacitor_SMD:C_0201_0603Metric
- D1: footprint (none) -> Diode_SMD:D_SMB
- L1, L2: footprint (none) -> Inductor_SMD:L_0201_0603Metric
- P1: footprint (none) -> Connector_USB:USB_C_Receptacle_Amphenol_12401610E4-2A
- R_BOT1: renamed from R_BOT; footprint (none) -> Resistor_SMD:R_0201_0603Metric_Pad0.64x0.40mm_HandSolder
- R_EN_1, R_EN_2: footprint (none) -> Resistor_SMD:R_0201_0603Metric_Pad0.64x0.40mm_HandSolder
- R_GOOD1: renamed from R_GOOD; footprint (none) -> Resistor_SMD:R_0201_0603Metric_Pad0.64x0.40mm_HandSolder
- R_TOP1: renamed from R_TOP; footprint (none) -> Resistor_SMD:R_0603_1608Metric_Pad0.98x0.95mm_HandSolder
Connections:
- net +12V: now also C11.1, C27.1, C28.1, L3.2; no longer BAT_+1.1
- net GND: now also C11.2, C27.2, C28.2, C29.1, C30.2, C31.2, C32.1, C33.2, D4.1 (A1), Q7.4 (G)
- net HSE_I: now also C29.2, X1.2
- net HSE_O: now also C31.1, X1.1
- net LSE_I: now also C32.2, X2.2
- net LSE_O: now also C33.1, X2.1
- net USART_RX: now also J5.2 (Pin_2)
- net USART_TX: now also J5.1 (Pin_1)
- new net: BAT_+1.1, D4.2 (A2), Q7.5 (D)
- new net: C30.1, L3.1, Q7.1 (S), Q7.2 (S), Q7.3 (S)
- no-connect marks 0 -> 14
Other:
- moved on the sheet: BAT_+1
