File: BLDC_Testboard/untitled.kicad_sch (KiCad schematic)
At the start: 36 parts, among them J2 Conn_01x01_Pin, J3 Conn_01x01_Pin, J4 Conn_01x01_Pin, Q1 CSD17578Q5A, Q2 CSD17578Q5A, Q3 CSD17578Q5A, Q4 CSD17578Q5A, Q5 CSD17578Q5A, Q6 CSD17578Q5A, U4 DRV8302DCA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

Commit message: Add files via upload
Parts:
- C12, C13, C14, C15, C16, C17, C18, C19, C20, C21, C22, C23: footprint (none) -> Capacitor_SMD:C_0201_0603Metric
- R1, R2, R3, R4, R5, R6, R7, R8, R9: footprint (none) -> Resistor_SMD:R_0201_0603Metric_Pad0.64x0.40mm_HandSolder
- R_Shunt_B1: renamed from R_Shunt_B; footprint (none) -> Resistor_SMD:R_0603_1608Metric_Pad0.98x0.95mm_HandSolder
- R_Shunt_c1: renamed from R_Shunt_c; footprint (none) -> Resistor_SMD:R_0603_1608Metric_Pad0.98x0.95mm_HandSolder
- U4: footprint DCA56_6P35X3P61 -> DRV8302:DCA56_6P35X3P61
Connections:
- net Current_SP1- is gone; now on net GND: U4.32 (SP1)
- net Current_SP2- is gone; now on net GND: U4.30 (SP2)
- net PH_SL_B is gone; now on net Current_SN1+: Q4.1 (S), Q4.2 (S), Q4.3 (S), R_Shunt_B1.1, U4.39 (SL_B)
- net PH_SL_C is gone; now on net Current_SN2+: Q6.1 (S), Q6.2 (S), Q6.3 (S), R_Shunt_c1.1, U4.34 (SL_C)
- net GND: no longer U4.57 (EPAD)
